File: Test1/Test1.sch (KiCad schematic (older format))
At the start: 74 parts, among them J1 Screw_Terminal_01x03, J2 Screw_Terminal_01x03, J3 Screw_Terminal_01x03, J4 Screw_Terminal_01x03, J5 Screw_Terminal_01x03, J6 Screw_Terminal_01x03, J7 Screw_Terminal_01x03, J8 Screw_Terminal_01x03, Q1 BC337, Q2 BC337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

Commit message: Se agrega PCB Layout
Falta rutear
Parts:
- added JPSWPUERTA1: Jumper_3_Open, Connector_PinHeader_2.54mm:PinHeader_1x03_P2.54mm_Vertical, symbol Jumper:Jumper_3_Open
- JUSB1: footprint Connector_PinSocket_2.00mm:PinSocket_1x06_P2.00mm_Vertical -> Connector_PinSocket_2.54mm:PinSocket_1x06_P2.54mm_Vertical
- renumbered SWPuertaNC1 to SWPanel1
Connections:
- net +5V: now also JPConf&Supply1.2 (C), JizqMDOT1.1 (Pin_1), JPSWPUERTA1.1 (A)
- net AI7: now also JizqMDOT1.2 (Pin_2); no longer JderMDOT1.9 (Pin_9)
- net DIPuerta: now also JderMDOT1.9 (Pin_9)
- net 5VUSB: now reaches JUSB1.1 (Pin_1)
- net 5VUSB: now also JPConf&Supply1.1 (A)
- net 3.3VMdot renamed 3VMdot
- net 3VMdot: now also JPSWPUERTA1.3 (B); no longer SWPanel1.2, SWPanel1.4
- net 3.3VUSB: no longer names the net of JUSB1.6 (Pin_6)
- net 3.3VUSB: no longer JPConf&Supply1.1 (A)
- new net: JPSWPUERTA1.2 (C), SWPanel1.2, SWPanel1.4
- no-connect marks 7 -> 9
Changed lines of the file:
@@
 	14750 8000 13950 8000
 Wire Wire Line
-	13800 7750 13800 7300
+	13800 7750 13800 7400
 Text GLabel 13800 7300 1    50   Input ~ 0
 Vreg5V
@@
 F 0 "JUSB1" V 15496 11348 50  0000 L CNN
 F 1 "Conn_01x06_Female" V 15587 11348 50  0000 L CNN
-F 2 "Connector_PinSocket_2.00mm:PinSocket_1x06_P2.00mm_Vertical" H 15650 11100 50  0001 C CNN
+F 2 "Connector_PinSocket_2.54mm:PinSocket_1x06_P2.54mm_Vertical" H 15650 11100 50  0001 C CNN
 F 3 "~" H 15650 11100 50  0001 C CNN
 	1    15650 11100
@@
 	13800 10250 13800 8250
 Wire Wire Line
-	13800 10250 15350 10250
-Wire Wire Line
-	15350 10250 15350 10900
-Wire Wire Line
 	15750 10500 15250 10500
 Connection ~ 15250 10500
@@
 	13500 10250 13500 10050
 Connection ~ 13500 10050
-Wire Wire Line
-	13500 10050 14400 10050
 $Comp
 L Device:R RModo1
@@
 	13700 8800 13700 8400
 Text GLabel 14950 10050 1    50   Input ~ 0
-3.3VMdot
+3VMdot
 Text GLabel 13800 9450 2    50   Input ~ 0
-3.3VUSB
+5VUSB
 $Comp
 L Connector:Conn_01x10_Female JderMDOT1
@@
 Text GLabel 16900 8700 2    50   Input ~ 0
 DO1
-Text GLabel 16900 8800 2    50   Input ~ 0
+Text GLabel 14250 8100 0    50   Input ~ 0
 AI7
 Text GLabel 16900 8900 2    50   Input ~ 0
@@
 	12450 7600 12600 7600
 Wire Wire Line
-	12600 7600 12600 7450
-Wire Wire Line
 	11650 8300 11650 9000
 Wire Wire Line
@@
 Wire Wire Line
 	12650 8300 14750 8300
-Wire Wire Line
-	12600 7450 14400 7450
-Wire Wire Line
-	14400 7450 14400 10050
-Connection ~ 14400 10050
-Wire Wire Line
-	14400 10050 15150 10050
 Wire Wire Line
 	11650 7800 12050 7800
@@
 Wire Wire Line
 	12450 7400 12600 7400
-Wire Wire Line
-	12600 7400 12600 7450
-Connection ~ 12600 7450
 NoConn ~ 15350 9400
 NoConn ~ 15450 9400
@@
 NoConn ~ 16200 8600
 NoConn ~ 15450 10900
-NoConn ~ 15850 10900
+NoConn ~ 15350 10900
 Wire Wire Line
 	15750 10500 15750 10900
@@
 	1    0    0    -1
 $EndComp
-Text GLabel 21100 1300 2    50   Input ~ 0
-Vreg5V
 $Comp
 L Transistor_BJT:BC337 Q2
@@
 	1    0    0    -1
 $EndComp
-Text GLabel 19000 1300 2    50   Input ~ 0
-Vreg5V
 $Comp
 L Transistor_BJT:BC337 Q3
@@
 	1    0    0    -1
 $EndComp
-Text GLabel 16700 1250 2    50   Input ~ 0
-Vreg5V
 Text GLabel 17800 2350 0    50   Input ~ 0
 DO2
@@
 DO1
 $Comp
-L Switch:SW_Push_Open_Dual SWPuertaNC1
+L Switch:SW_Push_Open_Dual SWPanel1
 U 1 1 617A3C9D
 P 12250 7400
-F 0 "SWPuertaNC1" H 12250 7610 50  0000 C CNN
+F 0 "SWPanel1" H 12250 7610 50  0000 C CNN
 F 1 "SW_Push_Open_Dual" H 12250 7519 50  0000 C CNN
 F 2 "TerminalBlock_Phoenix:TerminalBlock_Phoenix_MKDS-1,5-2_1x02_P5.00mm_Horizontal" H 12250 7600 50  0001 C CNN
@@
 	1    0    0    -1
 $EndComp
+Wire Wire Line
+	13500 10050 13650 10050
+Wire Wire Line
+	12600 7400 12600 7600
+Wire Wire Line
+	12600 7400 12850 7400
+Connection ~ 12600 7400
+Connection ~ 13800 7400
+Wire Wire Line
+	13800 7400 13800 7300
+Wire Wire Line
+	14250 8100 14750 8100
+Text GLabel 16900 8800 2    50   Input ~ 0
+DIPuerta
+Wire Wire Line
+	15850 10250 15850 10900
+Wire Wire Line
+	13800 10250 15850 10250
+Text GLabel 14450 8000 1    50   Input ~ 0
+VccMDOT
+Text GLabel 16700 1250 2    50   Input ~ 0
+VccMDOT
+Text GLabel 19000 1300 2    50   Input ~ 0
+VccMDOT
+Text GLabel 21100 1300 2    50   Input ~ 0
+VccMDOT
+$Comp
+L Jumper:Jumper_3_Open JPSWPUERTA1
+U 1 1 6128AE99
+P 13000 7400
+F 0 "JPSWPUERTA1" V 12954 7487 50  0000 L CNN
+F 1 "Jumper_3_Open" V 13045 7487 50  0000 L CNN
+F 2 "Connector_PinHeader_2.54mm:PinHeader_1x03_P2.54mm_Vertical" H 13000 7400 50  0001 C CNN
+F 3 "~" H 13000 7400 50  0001 C CNN
+	1    13000 7400
+	0    1    1    0
+$EndComp
+Wire Wire Line
+	13350 7400 13800 7400
+Wire Wire Line
+	13350 7400 13350 7150
+Wire Wire Line
+	13350 7150 13000 7150
+Wire Wire Line
+	13000 7650 13000 7800
+Wire Wire Line
+	13000 7800 12750 7800
+Wire Wire Line
+	12750 7800 12750 9500
+Wire Wire Line
+	12750 9500 13650 9500
+Wire Wire Line
+	13650 9500 13650 10050
+Connection ~ 13650 10050
+Wire Wire Line
+	13650 10050 15150 10050
+NoConn ~ 14750 8700
+NoConn ~ 14750 8800
 $EndSCHEMATC

Commit message: Cambios antes de comenzar a rutear
Se modificaron algunas cosas en esquemático para comenzar a rutear.
Connections:
- net 3VMdot is gone; now on net +3V3: JPSWPUERTA1.3 (B), JabajoMDOT1.8 (Pin_8), SWModo1.2, SWModo1.4
Changed lines of the file:
@@
 NoConn ~ 14750 8700
 NoConn ~ 14750 8800
+Text GLabel 4950 8150 1    50   Input ~ 0
+3VMdot
+Text GLabel 2550 8150 1    50   Input ~ 0
+3VMdot
+Text GLabel 2550 5750 1    50   Input ~ 0
+3VMdot
+Text GLabel 4950 5750 1    50   Input ~ 0
+3VMdot
+Text GLabel 2550 3400 1    50   Input ~ 0
+3VMdot
+Text GLabel 4950 3400 1    50   Input ~ 0
+3VMdot
+Text GLabel 2550 1000 1    50   Input ~ 0
+3VMdot
+Text GLabel 4950 1000 1    50   Input ~ 0
+3VMdot
 $EndSCHEMATC

Commit message: Hasta acá se arreglaron los problemas de K
Funciona todo, envía ok, tanto caudal como frecuencia y se despierta si hay un cable cortado. Calcula correctamente y se puede configurar por usb. Falta probar panel conectado y luego la batería.
Parts:
- Dreg1, Dreg2: footprint Diode_THT:D_A-405_P12.70mm_Horizontal -> Diode_THT:D_DO-15_P15.24mm_Horizontal
Changed lines of the file:
@@
 F 0 "Dreg1" V 9654 2380 50  0000 L CNN
 F 1 "D_Zener" V 9745 2380 50  0000 L CNN
-F 2 "Diode_THT:D_A-405_P12.70mm_Horizontal" H 9700 2300 50  0001 C CNN
+F 2 "Diode_THT:D_DO-15_P15.24mm_Horizontal" H 9700 2300 50  0001 C CNN
 F 3 "~" H 9700 2300 50  0001 C CNN
 	1    9700 2300
@@
 F 0 "Dreg2" V 9954 5380 50  0000 L CNN
 F 1 "D_Zener" V 10045 5380 50  0000 L CNN
-F 2 "Diode_THT:D_A-405_P12.70mm_Horizontal" H 10000 5300 50  0001 C CNN
+F 2 "Diode_THT:D_DO-15_P15.24mm_Horizontal" H 10000 5300 50  0001 C CNN
 F 3 "~" H 10000 5300 50  0001 C CNN
 	1    10000 5300
